File: current/MRR_ESPE.sch (KiCad schematic (older format))
At the start: 166 parts, among them J1 X_MIN, J10 PART_FAN, J11 UNUSED, J12 T_BED, J13 T_E0, J14 I2C/SPI, J15 AUX1, J16 USB_B_Micro, J17 E0_FAN, J18 CASE_FAN, J19 E1_FAN, J2 Z_MIN, J20 CS_PINS, J21 X_MOTOR, J22 Z_MOTOR, J23 Y_MOTOR, J24 E0_MOTOR, J25 E1_MOTOR, J26 EXP3, J3 BED, J4 Micro_SD_Card_China, J5 Y_MIN, J6 Z_PROBE, J7 E0, J8 T_E0, J9 PWR_IN, Q1 IRLS3034PBF, Q2 IRLR8743TRPBF, Q3 WST3392, Q4 S9014, Q5 S9014, Q6 WST3392, SW1 RESET, U1 ESP32-WROOM-32D, U10 TLP182, U11 Pololu_board, U13 74HC595, U14 74HC595, U15 74HC595, U2 TPS54340DDA, U3 CH340C, U4 AMS1117-3.3, U5 Pololu_board, U6 Pololu_board, U7 74HC595, U8 Pololu_board, U9 Pololu_board

Commit message: Added v0.5
Parts:
- removed JP28: VUSB_EN, Connector_PinHeader_2.54mm:PinHeader_1x02_P2.54mm_Vertical, symbol Device:Jumper
- added C28: 100nF25V, Capacitor_SMD:C_0805_2012Metric, symbol Device:C
- added JP28: 5V_SEL, Connector_PinHeader_2.54mm:PinHeader_1x03_P2.54mm_Vertical, symbol Jumper:Jumper_3_Open
- added JP30: PWR_SEL, Connector_PinHeader_2.54mm:PinHeader_1x03_P2.54mm_Vertical, symbol Jumper:Jumper_3_Open
- C1, C2, C20, C21, C23, C24, C25, C3: value 100nF16V -> 100nF25V; LCSC Part Number (none) -> C128353; Manufacturer (none) -> Walsin Tech Corp; Mfg part no. (none) -> 0805B104K250
- C10: LCSC Part Number (none) -> C161260; Manufacturer (none) -> Murata Electronics; Mfg part no. (none) -> GCM21BR71H104KA37L
- C11: LCSC Part Number (none) -> C52278; Manufacturer (none) -> Guangdong Fenghua Advanced Tech; Mfg part no. (none) -> 0805B103K500NT
- C12: value 47uF16V -> 47uF10V; LCSC Part Number (none) -> C92821; Manufacturer (none) -> Taiyo Yuden; Mfg part no. (none) -> LMK316BJ476ML-T
- C13, C14: value 10uF16V -> 47uF6.3V; LCSC Part Number (none) -> C87159; Manufacturer (none) -> Taiyo Yuden; Mfg part no. (none) -> JMK212BJ476MG-T
- C15, C16, C17, C18, C27: LCSC Part Number (none) -> C97811; Manufacturer (none) -> Semtech; Mfg part no. (none) -> CS1V101M-CRE77
- C19: value 100uF10V -> 100uF6.3V; LCSC Part Number (none) -> C15008; Manufacturer (none) -> Samsung Electro-Mechanics; Mfg part no. (none) -> CL31A107MQHNNNE
- C22: value 10uF16V -> 22uF6.3V; LCSC Part Number (none) -> C5674; Manufacturer (none) -> Samsung Electro-Mechanics; Mfg part no. (none) -> CL21A226MQQNNNE
- C26, C5, C6: value 22uF10V -> 22uF6.3V; LCSC Part Number (none) -> C5674; Manufacturer (none) -> Samsung Electro-Mechanics; Mfg part no. (none) -> CL21A226MQQNNNE
- C4: LCSC Part Number (none) -> C176665; Manufacturer (none) -> Lelon; Mfg part no. (none) -> VEJ101M1HTR-0810
- C7: LCSC Part Number (none) -> C307575; Manufacturer (none) -> Samsung Electro-Mechanics; Mfg part no. (none) -> CL31B475KBHNFNE
- C8: LCSC Part Number (none) -> C152862; Manufacturer (none) -> Walsin Tech Corp; Mfg part no. (none) -> 0805B821K500CT
- C9: LCSC Part Number (none) -> C296102; Manufacturer (none) -> Walsin Tech Corp; Mfg part no. (none) -> 0805N560J500CT
- D1, D3: LCSC Part Number (none) -> C72037; Manufacturer (none) -> Everlight Elec; Mfg part no. (none) -> 17-21SURC/S530-A3/TR8
- D10, D11: LCSC Part Number (none) -> C73548; Manufacturer (none) -> Everlight Elec; Mfg part no. (none) -> 17-21SYGC/S530-E2/TR8
- D12, D13: LCSC Part Number (none) -> C72035; Manufacturer (none) -> Everlight Elec; Mfg part no. (none) -> 17-21/BHC-XL2M2TY/3T
- D14, D15: value 1N5819 -> 1N5819W; LCSC Part Number (none) -> C169540; Manufacturer (none) -> Shandong Jingdao Microelectronics; Mfg part no. (none) -> 1N5819W
- D2: LCSC Part Number (none) -> C81598; Manufacturer (none) -> Semtech; Mfg part no. (none) -> 1N4148W
- D4, D5: value 1N4007 -> 1N4007W; LCSC Part Number (none) -> C108803; Manufacturer (none) -> Shandong Jingdao Microelectronics; Mfg part no. (none) -> 1N4007W
- D7, D8: LCSC Part Number (none) -> C19224; Manufacturer (none) -> Nexperia; Mfg part no. (none) -> PESD5V0S1BA,115
- D9: LCSC Part Number (none) -> C72264; Manufacturer (none) -> Diodes Incorporated; Mfg part no. (none) -> B540C-13-F
- F1: value 20A 1808 -> 15A 2410; LCSC Part Number (none) -> C44480; Manufacturer (none) -> Littelfuse; Mfg part no. (none) -> 0451015.MRL
- F2: LCSC Part Number (none) -> C187558; Manufacturer (none) -> Littelfuse; Mfg part no. (none) -> 0456030.ER
- J1, J2, J5, J6: footprint Connector_PinHeader_2.54mm:PinHeader_1x03_P2.54mm_Vertical -> Connector_JST:JST_XH_B03B-XH-A_1x03_P2.50mm_Vertical; LCSC Part Number (none) -> C144394; Manufacturer (none) -> JST Sales America; Mfg part no. (none) -> B3B-XH-A(LF)(SN)
- J10, J12, J13, J18, JP17, JP23, JP29: LCSC Part Number (none) -> C124375; Manufacturer (none) -> Shenzhen Cankemeng; Mfg part no. (none) -> C124375
- J11, J14: LCSC Part Number (none) -> C124387; Manufacturer (none) -> Shenzhen Cankemeng; Mfg part no. (none) -> C124387
- J15: LCSC Part Number (none) -> C9135; Manufacturer (none) -> Boom Precision Elec; Mfg part no. (none) -> C9135
- J16: LCSC Part Number (none) -> C136000; Manufacturer (none) -> MOLEX; Mfg part no. (none) -> 105017-0001
- J17: value E0_FAN -> HS_FAN; LCSC Part Number (none) -> C124375; Manufacturer (none) -> Shenzhen Cankemeng; Mfg part no. (none) -> C124375
- J19: value E1_FAN -> EXT_FAN; LCSC Part Number (none) -> C124375; Manufacturer (none) -> Shenzhen Cankemeng; Mfg part no. (none) -> C124375
- J20: LCSC Part Number (none) -> C124379; Manufacturer (none) -> Shenzhen Cankemeng; Mfg part no. (none) -> C124379
- J21, J23, J24, J25: LCSC Part Number (none) -> C124378; Manufacturer (none) -> Shenzhen Cankemeng; Mfg part no. (none) -> C124378
- J22: LCSC Part Number (none) -> C124386; Manufacturer (none) -> Shenzhen Cankemeng; Mfg part no. (none) -> C124386
- J26: LCSC Part Number (none) -> C5665; Manufacturer (none) -> Boom Precision Elec; Mfg part no. (none) -> C5665
- J3: LCSC Part Number (none) -> C89120; Manufacturer (none) -> Phoenix Contact; Mfg part no. (none) -> MKDS3/2-5.08
- J4: LCSC Part Number (none) -> C111196; Manufacturer (none) -> SOFNG; Mfg part no. (none) -> TF-15×15
- J7: LCSC Part Number (none) -> C91153; Manufacturer (none) -> Phoenix Contact; Mfg part no. (none) -> MKDSN1.5/2-5.08
- J8: value T_E0 -> T_EXT; LCSC Part Number (none) -> C124375; Manufacturer (none) -> Shenzhen Cankemeng; Mfg part no. (none) -> C124375
- J9: LCSC Part Number (none) -> C90087; Manufacturer (none) -> Phoenix Contact; Mfg part no. (none) -> MKDS3/4-5.08
- JP1, JP10, JP11, JP12, JP13, JP14, JP15, JP16, JP18, JP19, JP2, JP20, JP22, JP25, JP26, JP27, JP3, JP4, JP5, JP6, JP7, JP8, JP9: LCSC Part Number (none) -> C124376; Manufacturer (none) -> Shenzhen Cankemeng; Mfg part no. (none) -> C124376
- JP21: value E0_ON -> HS_ON; LCSC Part Number (none) -> C124375; Manufacturer (none) -> Shenzhen Cankemeng; Mfg part no. (none) -> C124375
- JP24: value E1_ON -> EXT_ON; LCSC Part Number (none) -> C124375; Manufacturer (none) -> Shenzhen Cankemeng; Mfg part no. (none) -> C124375
- L1: LCSC Part Number (none) -> C181722; Manufacturer (none) -> Shun Xiang Nuo Elec; Mfg part no. (none) -> SMMS0530-4R7M
- Q3, Q6: LCSC Part Number (none) -> C148366; Manufacturer (none) -> Winsok Semicon; Mfg part no. (none) -> WST3392
- Q4, Q5: LCSC Part Number (none) -> C181164; Manufacturer (none) -> Guangdong Hottech; Mfg part no. (none) -> S9014
- R1, R3, R32, R33, R37, R39, R4, R41, R8: LCSC Part Number (none) -> C38522; Manufacturer (none) -> Uniroyal Elec; Mfg part no. (none) -> 0805W8F1002T5E
- R10, R12, R13, R40, R6: LCSC Part Number (none) -> C17415; Manufacturer (none) -> Uniroyal Elec; Mfg part no. (none) -> 0805W8F100JT5E
- R11, R14, R34, R42, R7: LCSC Part Number (none) -> C149504; Manufacturer (none) -> Uniroyal Elec; Mfg part no. (none) -> 0805W8F1003T5E
- R15, R22, R23: LCSC Part Number (none) -> C17444; Manufacturer (none) -> Uniroyal Elec; Mfg part no. (none) -> 0805W8F1202T5E
- R16, R17, R19, R2, R20: LCSC Part Number (none) -> C17673; Manufacturer (none) -> Uniroyal Elec; Mfg part no. (none) -> 0805W8F4701T5E
- R18: LCSC Part Number (none) -> C170958; Manufacturer (none) -> Walsin Tech Corp; Mfg part no. (none) -> WR08X7322FTL
- R21: LCSC Part Number (none) -> C170848; Manufacturer (none) -> Walsin Tech Corp; Mfg part no. (none) -> WR08X2372FTL
- R24: LCSC Part Number (none) -> C273994; Manufacturer (none) -> YAGEO; Mfg part no. (none) -> RC0805FR-0760K4L
- R25: LCSC Part Number (none) -> C17418; Manufacturer (none) -> Uniroyal Elec; Mfg part no. (none) -> 0805W8F1152T5E
- R26, R27: LCSC Part Number (none) -> C17477; Manufacturer (none) -> Uniroyal Elec; Mfg part no. (none) -> 0805W8F0000T5E
- R28: LCSC Part Number (none) -> C17557; Manufacturer (none) -> Uniroyal Elec; Mfg part no. (none) -> 0805W8F2200T5E
- R29, R36: LCSC Part Number (none) -> C17630; Manufacturer (none) -> Uniroyal Elec; Mfg part no. (none) -> 0805W8F3300T5E
- R30, R31, R5, R9: LCSC Part Number (none) -> C17520; Manufacturer (none) -> Uniroyal Elec; Mfg part no. (none) -> 0805W8F2201T5E
- R35, R38: LCSC Part Number (none) -> C17513; Manufacturer (none) -> Uniroyal Elec; Mfg part no. (none) -> 0805W8F1001T5E
- SW1: LCSC Part Number (none) -> C83206; Manufacturer (none) -> Korean Hroparts Elec; Mfg part no. (none) -> K2-6639SP-C4SC-04
- U1: LCSC Part Number (none) -> C95209; Manufacturer (none) -> Espressif Systems; Mfg part no. (none) -> ESP32-WROOM-32
- U10: LCSC Part Number (none) -> C96457; Manufacturer (none) -> TOSHIBA; Mfg part no. (none) -> TLP182(GB-TPL,E
- U11, U5, U6, U8, U9: LCSC Part Number (none) -> C27438; Manufacturer (none) -> Boom Precision Elec; Mfg part no. (none) -> x2
- U13, U14, U15, U7: value 74HC595 -> 74HCT595; footprint Package_SO:SOIC-16_3.9x9.9mm_P1.27mm -> Package_SO:TSSOP-16_4.4x5mm_P0.65mm; LCSC Part Number (none) -> C152276; Manufacturer (none) -> ON Semicon; Mfg part no. (none) -> MC74HCT595ADTR2G
- U2: LCSC Part Number (none) -> C45886; Manufacturer (none) -> Texas Instruments; Mfg part no. (none) -> TPS54340DDAR
- U3: LCSC Part Number (none) -> C84681; Manufacturer (none) -> Jiangsu Qin Heng; Mfg part no. (none) -> CH340C
- U4: LCSC Part Number (none) -> C6186; Manufacturer (none) -> Advanced Monolithic Systems; Mfg part no. (none) -> AMS1117-3.3
Connections:
- wire segments 358 -> 357
Other:
- note added: "Extra fan"
- note added: "Heat sink fan"
- note removed: "E0 fan"
- note removed: "E1 fan"
- moved on the sheet: D15

Commit message: Added v0.5rev1 to fix AUX1 issue
Changed lines of the file:
@@
 Sheet 1 1
 Title "MRR ESPE"
-Date "2019-10-06"
-Rev "v0.5"
+Date "2019-12-09"
+Rev "v0.5rev1"
 Comp ""
 Comment1 ""
@@
 	5400 3000 5400 2800
 Connection ~ 5400 2800
-Text GLabel 4750 8650 2    50   BiDi ~ 0
-UART-
 Text GLabel 4750 8750 2    50   BiDi ~ 0
+UART-
+Text GLabel 4750 8650 2    50   BiDi ~ 0
 UART+
 $Comp
