File: old/v0.5/MRR_ESPE.kicad_pcb (KiCad board)
At the start: 2 copper layers, 102 x 102 mm, 168 parts, among them J1 X_MIN, J10 PART_FAN, J11 UNUSED, J12 T_BED, J13 T_E0, J14 I2C/SPI, J15 AUX1, J16 USB_B_Micro, J17 HS_FAN, J18 CASE_FAN, J19 EXT_FAN, J2 Z_MIN, J20 CS_PINS, J21 X_MOTOR, J22 Z_MOTOR, J23 Y_MOTOR, J24 E0_MOTOR, J25 E1_MOTOR, J26 EXP3, J3 BED, J4 Micro_SD_Card_China, J5 Y_MIN, J6 Z_PROBE, J7 E0, J8 T_EXT, J9 PWR_IN, Q1 IRLS3034PBF, Q2 IRLR8743TRPBF, Q3 WST3392, Q4 S9014, Q5 S9014, Q6 WST3392, SW1 RESET, U1 ESP32-WROOM-32D, U10 TLP182, U11 Pololu_board, U13 74HCT595, U14 74HCT595, U15 74HCT595, U2 TPS54340DDA, U3 CH340C, U4 AMS1117-3.3, U5 Pololu_board, U6 Pololu_board, U7 74HCT595, U8 Pololu_board, U9 Pololu_board

Commit message: Added v0.5rev1 to fix AUX1 issue
Parts:
- C1, C2, C20, C21, C23, C24, C25, C28, C3: value 100nF25V -> 100nF16V
- C12: value 47uF10V -> 47uF16V
- C13, C14: value 47uF6.3V -> 10uF16V
- C19: value 100uF6.3V -> 100uF10V
- C22: value 22uF6.3V -> 10uF16V
- D14, D15: value 1N5819W -> 1N5819
- D4, D5: value 1N4007W -> 1N4007
- F1: value 15A 2410 -> 20A 1808
- F2: footprint projfp:Littelfuse_0456 -> projfp:Littelfuse_456
- U13, U14, U15, U7: value 74HCT595 -> 74HC595
Connections:
- J15 pad 6: UART+ -> UART-
- J15 pad 8: UART- -> UART+
Routing:
- net UART-: track 49.8 -> 53.3 mm
- net UART+: track 50.6 -> 48.6 mm
Other:
- board text added: "MRR ESPE v0.5"
- board text added: "Version date: 2019-10-06"
- board text removed: "MRR ESPE v0.5rev1"
- board text removed: "Version date: 2019-12-09"
